File: Board/charge_controller.brd (EAGLE design)
At the start: 72.4 x 50.8 mm, 23 parts

Commit message: design changed
Parts:
- COM: device linear:DIL14 -> atick_linear:DIL14
- D1, D2: device diode:DO35-7 -> atick_diode:DO35-7
- T1, T2: device transistor:TO92-CBE -> atick_transistor:TO92-CBE
- ZEN: device diode:SOD81 -> atick_diode:SOD81
- moved T1 1.27 mm to (31.8, 11.4)
- renumbered CON to LOADED
Routing:
- net GND: track 55.5 -> 10.2 mm
- net N$2: track 20.2 -> 25.3 mm, vias 0 -> 2
- net N$14: track 152.8 -> 154.7 mm
- net N$3: track 10.7 -> 12.5 mm
- net N$8: track 5.08 -> 3.81 mm
- net N$4: track 15.8 -> 15.0 mm
- net N$10: track 88.2 -> 88.7 mm
