File: Schematic/charge_controller.sch (EAGLE design)
At the start: 23 parts

Commit message: design changed
Parts:
- COM: device linear:LM324N -> atick_linear:LM324N
- D1, D2: device diode:1N4148DO35-7 -> atick_diode:1N4148DO35-7
- T1, T2: device transistor:MPS2222A-NPN-TO92-CBE -> atick_transistor:BF393-NPN-TO92-CBE
- ZEN: device diode:BZD23 -> atick_diode:BZD23
- renumbered CON to LOADED
